Commit message: Add top cover parts to turtlebot

File: turtlebot_description/urdf/stacks/hexagons.urdf.xacro (robot description, xacro)
@@ -212,4 +212,12 @@
           <cylinder length="0.006" radius="0.170"/>
         </geometry>
+ 	<surface>
+          <friction>
+            <ode>
+              <mu>100.01</mu>
+              <mu2>100.01</mu2>
+            </ode>
+          </friction>
+        </surface>
       </collision>
       <inertial>
@@ -221,4 +229,55 @@
       </inertial>
     </link>
+    <joint name="top_cover1_joint" type="fixed">
+      <origin xyz="-0.155 0.0  0.43" rpy="0 0 0"/>
+      <parent link="${parent}"/>
+      <child link="top_cover1"/>
+    </joint>
+    <link name="top_cover1">
+     <collision name="collision">
+       <geometry>
+         <box size="0.01 0.16 0.06"/>
+       </geometry>
+     </collision>
+     <visual name="visual">
+       <geometry>
+         <box size="0.01 0.16 0.06"/>
+       </geometry>
+     </visual>
+   </link>
+   <joint name="top_cover2_joint" type="fixed">
+     <origin xyz="-0.09 -0.13  0.43" rpy="0 0 1.05"/>
+     <parent link="${parent}"/>
+     <child link="top_cover2"/>
+   </joint>
+   <link name="top_cover2">
+    <collision name="collision">
+      <geometry>
+        <box size="0.01 0.16 0.06"/>
+      </geometry>
+    </collision>
+    <visual name="visual">
+      <geometry>
+        <box size="0.01 0.16 0.06"/>
+      </geometry>
+    </visual>
+  </link>
+  <joint name="top_cover3_joint" type="fixed">
+    <origin xyz="-0.09 0.13  0.43" rpy="0 0 -1.05"/>
+    <parent link="${parent}"/>
+    <child link="top_cover3"/>
+  </joint>
+  <link name="top_cover3">
+   <collision name="collision">
+     <geometry>
+       <box size="0.01 0.16 0.06"/>
+     </geometry>
+   </collision>
+   <visual name="visual">
+     <geometry>
+       <box size="0.01 0.16 0.06"/>
+     </geometry>
+   </visual>
+  </link>
   </xacro:macro>
 </robot>
